Commit message: updated usn_seadrone model

File: usn_drone_gazebo/urdf/components/lidar.xacro (robot description, xacro)
@@ -5,7 +5,7 @@
                params = "type:='16_beam'
                          name
-                         x:=0.7 y:=0 z:=1.8
+                         x:=0.7 y:=0 z:=0.1
                          R:=0 P:=0 Y:=0
-                         post_Y:=0 post_z_from:=1.2965">
+                         post_Y:=0 post_z_from:=0">
     <xacro:if value="${type == '16_beam'}">
       <xacro:wamv_3d_lidar name="${name}"

File: usn_drone_gazebo/urdf/components/wamv_3d_lidar.xacro (robot description, xacro)
@@ -23,5 +23,5 @@
   -->
   <xacro:macro name="wamv_3d_lidar" params="name
-                                            x:=0.7 y:=0 z:=1.8
+                                            x:=0.7 y:=0 z:=0.05
                                             R:=0 P:=0 Y:=0
                                             post_Y:=0 post_z_from:=1.2965

File: usn_drone_gazebo/urdf/components/wamv_camera.xacro (robot description, xacro)
@@ -1,5 +1,5 @@
 <?xml version="1.0"?>
 <robot xmlns:xacro="http://ros.org/wiki/xacro">
-  <xacro:macro name="wamv_camera" params="name x:=0.5 y:=0 z:=1.5 post_z_from:=1.2965 R:=0 P:=0 Y:=0 post_Y:=0 visualize:=False">
+  <xacro:macro name="wamv_camera" params="name x:=0.5 y:=0 z:=0.1 post_z_from:=0 R:=0 P:=0 Y:=0 post_Y:=0 visualize:=False">
     <!-- Define length variables for link positioning -->
     <xacro:property name="platform_z" value="${post_z_from}"/>

File: usn_drone_gazebo/urdf/usn_drone_gazebo.urdf.xacro (robot description, xacro)
@@ -92,7 +92,7 @@
     <xacro:include filename="$(arg component_xacro_file)"/>
     <xacro:yaml_components />
-    <!-- Add CPU Cases -->
+    <!-- Add CPU Cases >
     <xacro:include filename="$(find wamv_description)/urdf/cpu_cases.xacro" />
-    <xacro:cpu_cases position="-0.15 0 1.53" orientation="0 0 0"/>
+    <xacro:cpu_cases position="-0.15 0 1.53" orientation="0 0 0"/-->
   </xacro:if>
   <!-- Otherwise, add sensors based on enable variables -->
@@ -128,7 +128,7 @@
     <!-- ==== VRX sensor configuration ==== -->
     <xacro:if value="$(arg vrx_sensors_enabled)">
-      <!-- Add CPU Cases -->
+      <!-- Add CPU Cases >
       <xacro:include filename="$(find wamv_description)/urdf/cpu_cases.xacro" />
-      <xacro:cpu_cases position="-0.15 0 1.53" orientation="0 0 0"/>
+      <xacro:cpu_cases position="-0.15 0 1.53" orientation="0 0 0"/-->
       <!-- Add a stereo camera pair -->
       <xacro:wamv_camera name="front_left_camera" y="0.1" x="0.75" P="${radians(15)}" />
@@ -137,13 +137,13 @@
       <xacro:wamv_camera name="middle_right_camera" y="-0.45" P="${radians(15)}" Y="${radians(-90)}" post_Y="${radians(-90)}" />
       <!-- Add simulated GPS -->
-      <xacro:wamv_gps name="gps_wamv" x="-0.85" />
+      <xacro:wamv_gps name="gps_wamv" x="-0.05" z="0.0" />
       <!-- Add Simulated IMU -->
-      <xacro:wamv_imu name="imu_wamv" y="-0.2" />
+      <xacro:wamv_imu name="imu_wamv" y="-0.2" z="0.0" />
       <!-- Add 3D LIDAR -->
-      <xacro:lidar name="lidar_wamv" type="16_beam"/>
+      <xacro:lidar name="lidar_wamv" type="16_beam" />
       <!-- Add pinger -->
       <xacro:wamv_pinger name="pinger" position="1.0 0 -1.0" />
-      <!-- Add ball shooter (default pitch angle: ~-60 deg) -->
-      <xacro:wamv_ball_shooter name="ball_shooter" x="0.54" y="0.30" z="1.296" pitch="-1.04"/>
+      <!-- Add ball shooter (default pitch angle: ~-60 deg) >
+      <xacro:wamv_ball_shooter name="ball_shooter" x="0.54" y="0.30" z="1.296" pitch="-1.04"/-->
     </xacro:if>
   </xacro:unless>

File: vrx_gazebo/worlds/example_course.world.xacro (robot description, xacro)
@@ -13,6 +13,6 @@
       <wind_objs>
         <wind_obj>
-          <name>wamv</name>
-          <link_name>wamv/base_link</link_name>
+          <name>usn_drone</name>
+          <link_name>usn_drone/base_link</link_name>
           <coeff_vector>.5 .5 .33</coeff_vector>
         </wind_obj>

File: vrx_gazebo/worlds/xacros/usv_wind_plugin.xacro (robot description, xacro)
@@ -3,8 +3,8 @@
   <xacro:macro name="usv_wind_gazebo"
                params="**wind_objs
-                         direction:=270
-                         mean_vel:=0
-                         var_gain:=0
-                         var_time:=2
+                         direction:=270.0
+                         mean_vel:=20.0
+                         var_gain:=20.0
+                         var_time:=2.0
                          seed:=''
                          ros_update_rate:=10
