Commit message: added robot localization

File: usn_drone_gazebo/urdf/components/wamv_imu.xacro (robot description, xacro)
@@ -1,5 +1,5 @@
 <?xml version="1.0"?>
 <robot xmlns:xacro="http://ros.org/wiki/xacro">
-  <xacro:macro name="wamv_imu" params="name:=imu x:=0.3 y:=0.5 z:=1.3 R:=0 P:=0 Y:=0 update_rate:=15">
+  <xacro:macro name="wamv_imu" params="name:=imu x:=0 y:=0 z:=0 R:=0 P:=0 Y:=0 update_rate:=15">
     <link name="${namespace}/${name}_link">
       <visual name="${name}_visual">>

File: usn_drone_gazebo/urdf/usn_drone_gazebo.urdf.xacro (robot description, xacro)
@@ -108,5 +108,5 @@
     <!-- Add Simulated IMU -->
     <xacro:if value="$(arg imu_enabled)">
-      <xacro:wamv_imu name="imu_wamv" y="-0.2" />
+      <xacro:wamv_imu name="imu_wamv" />
     </xacro:if>
     <!-- Add 3D LIDAR -->
@@ -134,17 +134,29 @@
       <xacro:wamv_camera name="front_left_camera" y="0.1" x="0.75" P="${radians(15)}" />
       <xacro:wamv_camera name="front_right_camera" y="-0.1" x="0.75" P="${radians(15)}" />
-      <!-- Add a camera facing right -->
-      <xacro:wamv_camera name="middle_right_camera" y="-0.45" P="${radians(15)}" Y="${radians(-90)}" post_Y="${radians(-90)}" />
+      <!-- Add a camera facing right >
+      <xacro:wamv_camera name="middle_right_camera" y="-0.45" P="${radians(15)}" Y="${radians(-90)}" post_Y="${radians(-90)}" /-->
       <!-- Add simulated GPS -->
-      <xacro:wamv_gps name="gps_wamv" x="-0.05" z="0.0" />
+      <xacro:wamv_gps name="gps_wamv" x="0.05" z="0.0" />
       <!-- Add Simulated IMU -->
-      <xacro:wamv_imu name="imu_wamv" y="-0.2" z="0.0" />
+      <xacro:wamv_imu name="imu_wamv" x="-0.05" z="0.0" />
       <!-- Add 3D LIDAR -->
       <xacro:lidar name="lidar_wamv" type="16_beam" />
-      <!-- Add pinger -->
-      <xacro:wamv_pinger name="pinger" position="1.0 0 -1.0" />
+      <!-- Add pinger >
+      <xacro:wamv_pinger name="pinger" position="1.0 0 -1.0" /-->
       <!-- Add ball shooter (default pitch angle: ~-60 deg) >
       <xacro:wamv_ball_shooter name="ball_shooter" x="0.54" y="0.30" z="1.296" pitch="-1.04"/-->
     </xacro:if>
   </xacro:unless>
+  <gazebo>
+    <plugin name="p3d_base_controller" filename="libgazebo_ros_p3d.so">
+      <alwaysOn>true</alwaysOn>
+      <updateRate>50.0</updateRate>
+      <bodyName>usn_drone/base_link</bodyName>
+      <topicName>ground_truth/state</topicName>
+      <gaussianNoise>0.01</gaussianNoise>
+      <frameName>world</frameName>
+      <xyzOffsets>0 0 0</xyzOffsets>
+      <rpyOffsets>0 0 0</rpyOffsets>
+    </plugin>
+  </gazebo>
 </robot>

File: vrx_gazebo/worlds/xacros/usv_wind_plugin.xacro (robot description, xacro)
@@ -3,7 +3,7 @@
   <xacro:macro name="usv_wind_gazebo"
                params="**wind_objs
-                         direction:=270.0
-                         mean_vel:=1
-                         var_gain:=5
+                         direction:=0
+                         mean_vel:= 3
+                         var_gain:=1
                          var_time:=2.0
                          seed:=''

File: wave_gazebo/world_models/ocean_waves/model.xacro (robot description, xacro)
@@ -17,7 +17,7 @@
 -->
 <world xmlns:xacro="http://ros.org/wiki/xacro">
-  <xacro:macro name="ocean_waves" params="gain:=0.3 period:=5
+  <xacro:macro name="ocean_waves" params="gain:=1 period:=3
                      direction_x:=1.0 direction_y:=0.0
-                     angle:=0.4 scale:=1.5">
+                     angle:=0.4 scale:=1">
   <model name='ocean_waves'>
     <static>true</static>
