Commit message: test new branch

File: usn_drone_gazebo/urdf/components/ball_shooter.xacro (robot description, xacro)
@@ -1,5 +1,5 @@
 <?xml version="1.0"?>
 <robot xmlns:xacro="http://ros.org/wiki/xacro">
-  <xacro:macro name="wamv_ball_shooter" params="name:='ball_shooter' frameId:='wamv/ball_shooter' x:=0.55 y:=0.35 z:=1.4 pitch:='0' yaw:='0'">
+  <xacro:macro name="usn_drone_ball_shooter" params="name:='ball_shooter' frameId:='usn_drone/ball_shooter' x:=0.55 y:=0.35 z:=1.4 pitch:='0' yaw:='0'">
     <link name="${namespace}/${name}_base_link">
       <visual name="${name}_base_visual">
@@ -64,5 +64,5 @@
           <model_name>blue_projectile</model_name>
           <link_name>link</link_name>
-          <frame>wamv/ball_shooter_launcher_link</frame>
+          <frame>usn_drone/ball_shooter_launcher_link</frame>
           <pose>0.14 0 0 0 0 0</pose>
         </projectile>

File: usn_drone_gazebo/urdf/components/lidar.xacro (robot description, xacro)
@@ -1,5 +1,5 @@
 <?xml version="1.0" encoding="UTF-8"?>
 <robot xmlns:xacro="http://ros.org/wiki/xacro">
-  <xacro:include filename="$(find wamv_gazebo)/urdf/components/wamv_3d_lidar.xacro"/>
+  <xacro:include filename="$(find usn_drone_gazebo)/urdf/components/usn_drone_3d_lidar.xacro"/>
   <xacro:macro name="lidar"
                params = "type:='16_beam'
@@ -9,5 +9,5 @@
                          post_Y:=0 post_z_from:=0">
     <xacro:if value="${type == '16_beam'}">
-      <xacro:wamv_3d_lidar name="${name}"
+      <xacro:usn_drone_3d_lidar name="${name}"
                            x="${x}" y="${y}" z="${z}"
                            R="${R}" P="${P}" Y="${Y}"
@@ -15,8 +15,8 @@
                            vertical_lasers="16"/>
       <!--specs for 16 beam lidar are implemented by default.
-          See wamv_3d_lidar for those-->
+          See usn_drone_3d_lidar for those-->
     </xacro:if>
     <xacro:if value="${type == '32_beam'}">
-      <xacro:wamv_3d_lidar name="${name}"
+      <xacro:usn_drone_3d_lidar name="${name}"
                            x="${x}" y="${y}" z="${z}"
                            R="${R}" P="${P}" Y="${Y}"

File: usn_drone_gazebo/urdf/macros.xacro (robot description, xacro)
@@ -4,14 +4,14 @@
        name="WAM-V">
        <!-- Include dynamics macros -->
-       <xacro:include filename="$(find usn_drone_gazebo)/urdf/dynamics/wamv_gazebo_dynamics_plugin.xacro" />
+       <xacro:include filename="$(find usn_drone_gazebo)/urdf/dynamics/usn_drone_gazebo_dynamics_plugin.xacro" />
        <!-- Include sensor macros -->
-       <xacro:include filename="$(find usn_drone_gazebo)/urdf/components/wamv_camera.xacro" />
-       <xacro:include filename="$(find usn_drone_gazebo)/urdf/components/wamv_gps.xacro" />
-       <xacro:include filename="$(find usn_drone_gazebo)/urdf/components/wamv_imu.xacro" />
-       <xacro:include filename="$(find usn_drone_gazebo)/urdf/components/wamv_planar_lidar.xacro" />
-       <xacro:include filename="$(find usn_drone_gazebo)/urdf/components/wamv_3d_lidar.xacro" />
+       <xacro:include filename="$(find usn_drone_gazebo)/urdf/components/usn_drone_camera.xacro" />
+       <xacro:include filename="$(find usn_drone_gazebo)/urdf/components/usn_drone_gps.xacro" />
+       <xacro:include filename="$(find usn_drone_gazebo)/urdf/components/usn_drone_imu.xacro" />
+       <xacro:include filename="$(find usn_drone_gazebo)/urdf/components/usn_drone_planar_lidar.xacro" />
+       <xacro:include filename="$(find usn_drone_gazebo)/urdf/components/usn_drone_3d_lidar.xacro" />
        <xacro:include filename="$(find usn_drone_gazebo)/urdf/components/lidar.xacro" />
-       <xacro:include filename="$(find usn_drone_gazebo)/urdf/components/wamv_p3d.xacro" />
-       <xacro:include filename="$(find usn_drone_gazebo)/urdf/components/wamv_pinger.xacro" />
+       <xacro:include filename="$(find usn_drone_gazebo)/urdf/components/usn_drone_p3d.xacro" />
+       <xacro:include filename="$(find usn_drone_gazebo)/urdf/components/usn_drone_pinger.xacro" />
        <!-- Include ball shooter macros -->
        <xacro:include filename="$(find usn_drone_gazebo)/urdf/components/ball_shooter.xacro" />

File: usn_drone_gazebo/urdf/usn_drone_gazebo.urdf.xacro (robot description, xacro)
@@ -36,5 +36,5 @@
   <xacro:include filename="$(find usn_drone_gazebo)/urdf/usn_drone_gazebo.xacro"/>
   <!-- === Batteries === >
-  <xacro:include filename="$(find wamv_description)/urdf/battery.xacro"/>
+  <xacro:include filename="$(find usn_drone_description)/urdf/battery.xacro"/>
   <xacro:battery prefix="left" position="0 1 0.45" orientation="0 0 0"/>
   <xacro:battery prefix="right" position="0 -1 0.45" orientation="0 0 0"/-->
@@ -42,5 +42,5 @@
   <!-- Use thruster yaml file if given -->
   <xacro:if value="$(arg yaml_thruster_generation)">
-    <xacro:wamv_gazebo thruster_layout="$(arg thruster_xacro_file)"/>
+    <xacro:usn_drone_gazebo thruster_layout="$(arg thruster_xacro_file)"/>
   </xacro:if>
   <!-- Otherwise, add thrusters based on thruster_config variable -->
@@ -49,13 +49,13 @@
     <!-- Default WAM-V with two aft thrusters -->
     <xacro:if value="${thruster_conf == 'H'}">
-       <xacro:wamv_gazebo thruster_layout="$(find wamv_gazebo)/urdf/thruster_layouts/wamv_aft_thrusters.xacro"/>
+       <xacro:usn_drone_gazebo thruster_layout="$(find usn_drone_gazebo)/urdf/thruster_layouts/usn_drone_aft_thrusters.xacro"/>
     </xacro:if>
-    <!-- WAMV with "T" thruster configuration -->
+    <!-- usn_drone with "T" thruster configuration -->
     <xacro:if value="${thruster_conf == 'T'}">
-      <xacro:wamv_gazebo thruster_layout="$(find wamv_gazebo)/urdf/thruster_layouts/wamv_t_thrusters.xacro"/>
+      <xacro:usn_drone_gazebo thruster_layout="$(find usn_drone_gazebo)/urdf/thruster_layouts/usn_drone_t_thrusters.xacro"/>
     </xacro:if>
-    <!-- WAMV with "X" thruster configuration -->
+    <!-- usn_drone with "X" thruster configuration -->
     <xacro:if value="${thruster_conf == 'X'}">
-      <xacro:wamv_gazebo thruster_layout="$(find wamv_gazebo)/urdf/thruster_layouts/wamv_x_thrusters.xacro"/>
+      <xacro:usn_drone_gazebo thruster_layout="$(find usn_drone_gazebo)/urdf/thruster_layouts/usn_drone_x_thrusters.xacro"/>
     </xacro:if>
   </xacro:unless>
@@ -63,8 +63,8 @@
   <xacro:if value="$(arg locked)">
     <gazebo>
-      <link name="wamv_external_link"/>
-      <joint name="wamv_external_pivot_joint" type="universal">
-        <parent>wamv::wamv/base_link</parent>
-        <child>wamv_external_link</child>
+      <link name="usn_drone_external_link"/>
+      <joint name="usn_drone_external_pivot_joint" type="universal">
+        <parent>usn_drone::usn_drone/base_link</parent>
+        <child>usn_drone_external_link</child>
         <axis>
           <xyz>1 0 0</xyz>
@@ -74,7 +74,7 @@
         </axis2>
       </joint>
-      <joint name="wamv_external_riser" type="prismatic">
+      <joint name="usn_drone_external_riser" type="prismatic">
         <parent>world</parent>
-        <child>wamv_external_link</child>
+        <child>usn_drone_external_link</child>
         <axis>
           <limit>
@@ -93,5 +93,5 @@
     <xacro:yaml_components />
     <!-- Add CPU Cases >
-    <xacro:include filename="$(find wamv_description)/urdf/cpu_cases.xacro" />
+    <xacro:include filename="$(find usn_drone_description)/urdf/cpu_cases.xacro" />
     <xacro:cpu_cases position="-0.15 0 1.53" orientation="0 0 0"/-->
   </xacro:if>
@@ -100,51 +100,63 @@
     <!-- Add a front camera -->
     <xacro:if value="$(arg camera_enabled)">
-      <xacro:wamv_camera name="front_camera" y="0.3" x="0.75" P="${radians(15)}" />
+      <xacro:usn_drone_camera name="front_camera" y="0.3" x="0.75" P="${radians(15)}" />
     </xacro:if>
     <!-- Add simulated GPS -->
     <xacro:if value="$(arg gps_enabled)">
-      <xacro:wamv_gps name="gps_wamv" x="-0.85" />
+      <xacro:usn_drone_gps name="gps_usn_drone" x="-0.85" />
     </xacro:if>
     <!-- Add Simulated IMU -->
     <xacro:if value="$(arg imu_enabled)">
-      <xacro:wamv_imu name="imu_wamv" y="-0.2" />
+      <xacro:usn_drone_imu name="imu_usn_drone" />
     </xacro:if>
     <!-- Add 3D LIDAR -->
     <xacro:if value="$(arg lidar_enabled)">
-      <xacro:lidar name="lidar_wamv" y="-0.3" type="16_beam"/>
+      <xacro:lidar name="lidar_usn_drone" y="-0.3" type="16_beam"/>
     </xacro:if>
     <!-- Add P3D ground truth -->
     <xacro:if value="$(arg ground_truth_enabled)">
-      <xacro:wamv_p3d name="p3d_wamv"/>
+      <xacro:usn_drone_p3d name="p3d_usn_drone"/>
     </xacro:if>
     <!-- Add pinger -->
     <xacro:if value="$(arg pinger_enabled)">
-      <xacro:wamv_pinger name="pinger" position="1.0 0 -1.0" />
+      <xacro:usn_drone_pinger name="pinger" position="1.0 0 -1.0" />
     </xacro:if>
     <!-- Add ball shooter (default pitch angle: ~-60 deg) -->
     <xacro:if value="$(arg ball_shooter_enabled)">
-      <xacro:wamv_ball_shooter name="ball_shooter" x="0.54" y="0.30" z="1.296" pitch="-1.04"/>
+      <xacro:usn_drone_ball_shooter name="ball_shooter" x="0.54" y="0.30" z="1.296" pitch="-1.04"/>
     </xacro:if>
     <!-- ==== VRX sensor configuration ==== -->
     <xacro:if value="$(arg vrx_sensors_enabled)">
       <!-- Add CPU Cases >
-      <xacro:include filename="$(find wamv_description)/urdf/cpu_cases.xacro" />
+      <xacro:include filename="$(find usn_drone_description)/urdf/cpu_cases.xacro" />
       <xacro:cpu_cases position="-0.15 0 1.53" orientation="0 0 0"/-->
       <!-- Add a stereo camera pair -->
-      <xacro:wamv_camera name="front_left_camera" y="0.1" x="0.75" P="${radians(15)}" />
-      <xacro:wamv_camera name="front_right_camera" y="-0.1" x="0.75" P="${radians(15)}" />
-      <!-- Add a camera facing right -->
-      <xacro:wamv_camera name="middle_right_camera" y="-0.45" P="${radians(15)}" Y="${radians(-90)}" post_Y="${radians(-90)}" />
+      <xacro:usn_drone_camera name="front_left_camera" y="0.1" x="0.75" P="${radians(15)}" />
+      <xacro:usn_drone_camera name="front_right_camera" y="-0.1" x="0.75" P="${radians(15)}" />
+      <!-- Add a camera facing right >
+      <xacro:usn_drone_camera name="middle_right_camera" y="-0.45" P="${radians(15)}" Y="${radians(-90)}" post_Y="${radians(-90)}" /-->
       <!-- Add simulated GPS -->
-      <xacro:wamv_gps name="gps_wamv" x="-0.05" z="0.0" />
+      <xacro:usn_drone_gps name="gps_usn_drone" x="0.05" z="0.0" />
       <!-- Add Simulated IMU -->
-      <xacro:wamv_imu name="imu_wamv" y="-0.2" z="0.0" />
+      <xacro:usn_drone_imu name="imu_usn_drone" x="-0.05" z="0.0" />
       <!-- Add 3D LIDAR -->
-      <xacro:lidar name="lidar_wamv" type="16_beam" />
-      <!-- Add pinger -->
-      <xacro:wamv_pinger name="pinger" position="1.0 0 -1.0" />
+      <xacro:lidar name="lidar_usn_drone" type="16_beam" />
+      <!-- Add pinger >
+      <xacro:usn_drone_pinger name="pinger" position="1.0 0 -1.0" /-->
       <!-- Add ball shooter (default pitch angle: ~-60 deg) >
-      <xacro:wamv_ball_shooter name="ball_shooter" x="0.54" y="0.30" z="1.296" pitch="-1.04"/-->
+      <xacro:usn_drone_ball_shooter name="ball_shooter" x="0.54" y="0.30" z="1.296" pitch="-1.04"/-->
     </xacro:if>
   </xacro:unless>
+  <gazebo>
+    <plugin name="p3d_base_controller" filename="libgazebo_ros_p3d.so">
+      <alwaysOn>true</alwaysOn>
+      <updateRate>50.0</updateRate>
+      <bodyName>usn_drone/base_link</bodyName>
+      <topicName>ground_truth/state</topicName>
+      <gaussianNoise>0.01</gaussianNoise>
+      <frameName>world</frameName>
+      <xyzOffsets>0 0 0</xyzOffsets>
+      <rpyOffsets>0 0 0</rpyOffsets>
+    </plugin>
+  </gazebo>
 </robot>

File: usn_drone_gazebo/urdf/usn_drone_gazebo.xacro (robot description, xacro)
@@ -4,11 +4,11 @@
   <xacro:include filename="$(find usn_drone_gazebo)/urdf/macros.xacro" />
   <!-- Macro to create a WAM-V with dyanmics plugins and a customizeable thruster layout -->
-  <xacro:macro  name="wamv_gazebo" params="thruster_layout">
+  <xacro:macro  name="usn_drone_gazebo" params="thruster_layout">
     <!-- Defines the base vehicle -->
-    <xacro:include filename="$(find usn_drone)/urdf/usn_drone.urdf.xacro" />
+    <xacro:include filename="$(find usn_drone_description)/urdf/usn_drone.urdf.xacro" />
     <!-- Thruster Layout -->
     <xacro:include filename="${thruster_layout}"/>
     <!-- Attach hydrodynamics plugin -->
-    <xacro:usv_dynamics_gazebo name="wamv_dynamics_plugin"/>
+    <xacro:usv_dynamics_gazebo name="usn_drone_dynamics_plugin"/>
   </xacro:macro>
 </robot>

File: vrx_gazebo/worlds/xacros/usv_wind_plugin.xacro (robot description, xacro)
@@ -3,7 +3,7 @@
   <xacro:macro name="usv_wind_gazebo"
                params="**wind_objs
-                         direction:=270.0
-                         mean_vel:=1
-                         var_gain:=5
+                         direction:=0
+                         mean_vel:= 0
+                         var_gain:=0
                          var_time:=2.0
                          seed:=''

File: wave_gazebo/world_models/ocean_waves/model.xacro (robot description, xacro)
@@ -17,7 +17,7 @@
 -->
 <world xmlns:xacro="http://ros.org/wiki/xacro">
-  <xacro:macro name="ocean_waves" params="gain:=0.3 period:=5
-                     direction_x:=1.0 direction_y:=0.0
-                     angle:=0.4 scale:=1.5">
+  <xacro:macro name="ocean_waves" params="gain:=0 period:=3
+                     direction_x:=0 direction_y:=0.0
+                     angle:=0.4 scale:=1">
   <model name='ocean_waves'>
     <static>true</static>
