Commit message: added depth camera

File: usn_drone_gazebo/urdf/components/usn_drone_camera.xacro (robot description, xacro)
@@ -129,42 +129,43 @@
     <!-- Gazebo camera setup -->
     <gazebo reference="${namespace}/${name}_link">
-      <sensor type="camera" name="${name}_sensor">
-        <update_rate>30.0</update_rate>
-	<xacro:if value="${visualize}">
-	  <visualize>true</visualize>
-	</xacro:if>
-        <camera name="${name}_camera">
-          <horizontal_fov>1.3962634</horizontal_fov>
+      <sensor name="camera" type="depth">
+        <update_rate>20</update_rate>
+        <camera>
+          <horizontal_fov>2.094396*2</horizontal_fov>
           <image>
-            <width>1280</width>
-            <height>720</height>
+            <width>1920</width>
+            <height>1080</height>
             <format>R8G8B8</format>
           </image>
           <clip>
             <near>0.05</near>
-            <far>300</far>
+            <far>3</far>
           </clip>
-          <noise>
-            <type>gaussian</type>
-            <!-- Noise is sampled independently per pixel on each frame.
-                 That pixel's noise value is added to each of its color
-                 channels, which at that point lie in the range [0,1]. -->
-            <mean>0.0</mean>
-            <stddev>0.007</stddev>
-          </noise>
         </camera>
-        <plugin name="camera_plugin_${name}" filename="libgazebo_ros_camera.so">
+        <plugin name="camera_plugin" filename="libgazebo_ros_openni_kinect.so">
+          <baseline>0.2</baseline>
           <alwaysOn>true</alwaysOn>
+          <!-- Keep this zero, update_rate in the parent <sensor> tag
+            will control the frame rate. -->
           <updateRate>0.0</updateRate>
-          <cameraName>${namespace}/${sensor_namespace}${camera_namespace}${name}</cameraName>
-          <imageTopicName>image_raw</imageTopicName>
-          <cameraInfoTopicName>camera_info</cameraInfoTopicName>
-          <frameName>${namespace}/${name}_link_optical</frameName>
-          <hackBaseline>0.07</hackBaseline>
-          <distortionK1>0.0</distortionK1>
-          <distortionK2>0.0</distortionK2>
-          <distortionK3>0.0</distortionK3>
-          <distortionT1>0.0</distortionT1>
-          <distortionT2>0.0</distortionT2>
+          <cameraName>camera_ir</cameraName>
+          <imageTopicName>/camera/color/image_raw</imageTopicName>
+          <cameraInfoTopicName>/camera/color/camera_info</cameraInfoTopicName>
+          <depthImageTopicName>/camera/depth/image_raw</depthImageTopicName>
+          <depthImageCameraInfoTopicName>/camera/depth/camera_info</depthImageCameraInfoTopicName>
+          <pointCloudTopicName>/camera/depth/points</pointCloudTopicName>
+          <frameName>usn_drone/front_left_camera_link_optical</frameName>
+          <pointCloudCutoff>0.5</pointCloudCutoff>
+          <pointCloudCutoffMax>3.0</pointCloudCutoffMax>
+          <distortionK1>0</distortionK1>
+          <distortionK2>0</distortionK2>
+          <distortionK3>0</distortionK3>
+          <distortionT1>0</distortionT1>
+          <distortionT2>0</distortionT2>
+          <CxPrime>0</CxPrime>
+          <Cx>0</Cx>
+          <Cy>0</Cy>
+          <focalLength>0</focalLength>
+          <hackBaseline>0</hackBaseline>
         </plugin>
       </sensor>

File: usn_drone_gazebo/urdf/usn_drone_gazebo.urdf.xacro (robot description, xacro)
@@ -15,4 +15,5 @@
   <xacro:arg name="thruster_namespace" default="thrusters/"/>
   <xacro:arg name="camera_namespace" default="cameras/"/>
+  <xacro:arg name="zed_namespace" default="zed/"/>
   <xacro:arg name="sensor_namespace" default="sensors/"/>
   <xacro:arg name="pinger_namespace" default="pingers/"/>
@@ -102,4 +103,5 @@
       <xacro:usn_drone_camera name="front_camera" y="0.3" x="0.75" P="${radians(15)}" />
     </xacro:if>
+    <!-- <xacro:usn_drone_camera name="zed" y="0" x="2" P="${radians(15)}" /> -->
     <!-- Add simulated GPS -->
     <xacro:if value="$(arg gps_enabled)">
@@ -133,5 +135,5 @@
       <!-- Add a stereo camera pair -->
       <xacro:usn_drone_camera name="front_left_camera" y="0.1" x="0.75" P="${radians(15)}" />
-      <xacro:usn_drone_camera name="front_right_camera" y="-0.1" x="0.75" P="${radians(15)}" />
+      <!-- <xacro:usn_drone_camera name="front_right_camera" y="-0.1" x="0.75" P="${radians(15)}" /> -->
       <!-- Add a camera facing right >
       <xacro:usn_drone_camera name="middle_right_camera" y="-0.45" P="${radians(15)}" Y="${radians(-90)}" post_Y="${radians(-90)}" /-->

File: wave_gazebo/world_models/ocean_waves/model.xacro (robot description, xacro)
@@ -17,7 +17,7 @@
 -->
 <world xmlns:xacro="http://ros.org/wiki/xacro">
-  <xacro:macro name="ocean_waves" params="gain:=0 period:=3
-                     direction_x:=0 direction_y:=0.0
-                     angle:=0.4 scale:=1">
+  <xacro:macro name="ocean_waves" params="gain:=0.1 period:=5
+                     direction_x:=1.0 direction_y:=0.0
+                     angle:=0.4 scale:=1.5">
   <model name='ocean_waves'>
     <static>true</static>
@@ -26,5 +26,5 @@
       <update_rate>30</update_rate>
       <size>1000 1000</size>
-      <cell_count>50 50</cell_count>
+      <cell_count>70 70</cell_count>
       <wave>
 				<model>PMS</model>

Commit message: modified mpc

File: usn_drone_gazebo/urdf/components/usn_drone_camera.xacro (robot description, xacro)
@@ -3,73 +3,60 @@
   <xacro:macro name="usn_drone_camera" params="name x:=0.5 y:=0 z:=0.1 post_z_from:=0 R:=0 P:=0 Y:=0 post_Y:=0 visualize:=False">
     <!-- Define length variables for link positioning -->
-    <xacro:property name="platform_z" value="${post_z_from}"/>
-    <xacro:property name="post_to_post_arm_x" value="0.03"/>
-    <xacro:property name="post_arm_to_camera_x" value="0.02"/>
-    <xacro:property name="post_arm_to_camera_z" value="0.027"/>
+    <xacro:property name="platform_z" value="${post_z_from}" />
+    <xacro:property name="post_to_post_arm_x" value="0.03" />
+    <xacro:property name="post_arm_to_camera_x" value="0.02" />
+    <xacro:property name="post_arm_to_camera_z" value="0.027" />
     <!-- Monocular Camera -->
     <link name="${namespace}/${name}_link">
       <visual name="${name}_visual">
-        <origin xyz="-0.033 0 0" rpy="0 0 ${pi/2}"/>
+        <origin xyz="-0.033 0 0" rpy="0 0 ${pi/2}" />
         <geometry>
-          <mesh filename="package://vrx_gazebo/models/mono_camera/mesh/mono_camera.dae"/>
+          <mesh filename="package://vrx_gazebo/models/mono_camera/mesh/mono_camera.dae" />
         </geometry>
       </visual>
       <collision name="${name}_lens_collision">
-        <origin xyz="0.018 0 0" rpy="0 ${pi/2} 0"/>
+        <origin xyz="0.018 0 0" rpy="0 ${pi/2} 0" />
         <geometry>
-          <cylinder radius="0.015" length="0.042"/>
+          <cylinder radius="0.015" length="0.042" />
         </geometry>
       </collision>
       <collision name="${name}_box_collision">
-        <origin xyz="-0.0205 0 0" rpy="0 0 0"/>
+        <origin xyz="-0.0205 0 0" rpy="0 0 0" />
         <geometry>
-          <box size="0.036 0.03 0.03"/>
+          <box size="0.036 0.03 0.03" />
         </geometry>
       </collision>
       <!-- Model inertia as box with <size>0.078 0.03 0.03</size> -->
       <inertial>
-        <mass value="0.3"/>
-        <inertia
-          ixx="0.0000450"
-          iyy="0.0001746"
-          izz="0.0001746"
-          ixy="0"
-          ixz="0"
-          iyz="0"/>
+        <mass value="0.3" />
+        <inertia ixx="0.0000450" iyy="0.0001746" izz="0.0001746" ixy="0" ixz="0" iyz="0" />
       </inertial>
     </link>
     <!-- Define a link for the optical frame.  This will match the sensor frame and
          be oriented in the camera convention. -->
-    <link name="${namespace}/${name}_link_optical">
-    </link>
+    <link name="${namespace}/${name}_link_optical"></link>
     <!-- Define post length and mass based on desired z position of sensor -->
-    <xacro:property name="post_length" value="${z-platform_z-post_arm_to_camera_z}"/>
-    <xacro:property name="post_mass_per_meter" value="0.9"/>
-    <xacro:property name="post_mass" value="${post_mass_per_meter * post_length}"/>
-    <xacro:property name="post_radius" value="0.0076"/>
+    <xacro:property name="post_length" value="${z-platform_z-post_arm_to_camera_z}" />
+    <xacro:property name="post_mass_per_meter" value="0.9" />
+    <xacro:property name="post_mass" value="${post_mass_per_meter * post_length}" />
+    <xacro:property name="post_radius" value="0.0076" />
     <!-- Sensor post -->
     <link name="${namespace}/${name}_post_link">
       <visual>
         <geometry>
-          <cylinder radius="${post_radius}" length="${post_length}"/>
+          <cylinder radius="${post_radius}" length="${post_length}" />
         </geometry>
         <material name="${name}_post_material">
-          <color rgba="0.0 0.0 0.0 1.0"/>
+          <color rgba="0.0 0.0 0.0 1.0" />
         </material>
       </visual>
       <collision name="${name}_post_collision">
         <geometry>
-          <cylinder radius="${post_radius}" length="${post_length}"/>
+          <cylinder radius="${post_radius}" length="${post_length}" />
         </geometry>
       </collision>
       <inertial>
-        <mass value="${post_mass}"/>
-        <inertia
-          ixx="${(post_mass/12) * (3*post_radius*post_radius + post_length*post_length)}"
-          iyy="${(post_mass/12) * (3*post_radius*post_radius + post_length*post_length)}"
-          izz="${(post_mass/2) * (post_radius*post_radius)}"
-          ixy="0"
-          ixz="0"
-          iyz="0"/>
+        <mass value="${post_mass}" />
+        <inertia ixx="${(post_mass/12) * (3*post_radius*post_radius + post_length*post_length)}" iyy="${(post_mass/12) * (3*post_radius*post_radius + post_length*post_length)}" izz="${(post_mass/2) * (post_radius*post_radius)}" ixy="0" ixz="0" iyz="0" />
       </inertial>
     </link>
@@ -77,30 +64,24 @@
     <link name="${namespace}/${name}_post_arm_link">
       <visual name="${name}_post_arm_visual">
-        <origin xyz="-0.038 0 -0.003" rpy="${radians(-60)} 0 ${-pi/2}"/>
+        <origin xyz="-0.038 0 -0.003" rpy="${radians(-60)} 0 ${-pi/2}" />
         <geometry>
-          <mesh filename="package://vrx_gazebo/models/sensor_post/mesh/sensor_post_arm.dae"/>
+          <mesh filename="package://vrx_gazebo/models/sensor_post/mesh/sensor_post_arm.dae" />
         </geometry>
       </visual>
       <collision name="${name}_post_arm_collision">
-        <origin xyz="0 0 0" rpy="${radians(-60)-pi/20} 0 ${-pi/2}"/>
+        <origin xyz="0 0 0" rpy="${radians(-60)-pi/20} 0 ${-pi/2}" />
         <geometry>
-          <cylinder radius="0.008" length="0.065"/>
+          <cylinder radius="0.008" length="0.065" />
         </geometry>
       </collision>
       <inertial>
-        <origin xyz="0 0 0" rpy="${radians(-60)-pi/20} 0 ${-pi/2}"/>
-        <mass value="0.1"/>
-        <inertia
-          ixx="0.00003680833"
-          iyy="0.00003680833"
-          izz="0.00000320000"
-          ixy="0"
-          ixz="0"
-          iyz="0"/>
+        <origin xyz="0 0 0" rpy="${radians(-60)-pi/20} 0 ${-pi/2}" />
+        <mass value="0.1" />
+        <inertia ixx="0.00003680833" iyy="0.00003680833" izz="0.00000320000" ixy="0" ixz="0" iyz="0" />
       </inertial>
     </link>
     <!-- Base to sensor post joint -->
-    <xacro:property name="post_z" value="${platform_z+post_length/2}"/>
-    <xacro:property name="post_to_camera_x" value="${post_to_post_arm_x+post_arm_to_camera_x}"/>
+    <xacro:property name="post_z" value="${platform_z+post_length/2}" />
+    <xacro:property name="post_to_camera_x" value="${post_to_post_arm_x+post_arm_to_camera_x}" />
     <joint name="${namespace}/base_to_${name}_post_joint" type="fixed">
       <origin xyz="${x-(post_to_camera_x)*cos(post_Y)} ${y-(post_to_camera_x)*sin(post_Y)} ${post_z}" rpy="0 0 ${post_Y}" />
@@ -155,5 +136,5 @@
           <depthImageCameraInfoTopicName>/camera/depth/camera_info</depthImageCameraInfoTopicName>
           <pointCloudTopicName>/camera/depth/points</pointCloudTopicName>
-          <frameName>usn_drone/front_left_camera_link_optical</frameName>
+          <frameName>usn_drone/front_camera_link_optical</frameName>
           <pointCloudCutoff>0.5</pointCloudCutoff>
           <pointCloudCutoffMax>3.0</pointCloudCutoffMax>

File: usn_drone_gazebo/urdf/thruster_layouts/usn_drone_gazebo_thruster_config.xacro (robot description, xacro)
@@ -1,5 +1,5 @@
 <?xml version="1.0"?>
 <plugin xmlns:xacro="http://ros.org/wiki/xacro">
-  <xacro:macro  name="usn_drone_gazebo_thruster_config" params="name enable_angle:=true">
+  <xacro:macro name="usn_drone_gazebo_thruster_config" params="name enable_angle:=true">
     <thruster>
       <!-- Required Parameters -->
@@ -12,6 +12,6 @@
       <!-- Optional Parameters -->
       <mappingType>1</mappingType>
-      <maxCmd>1.0</maxCmd>
-      <maxForceFwd>250.0</maxForceFwd>
+      <maxCmd>1</maxCmd>
+      <maxForceFwd>100</maxForceFwd>
       <maxForceRev>-100.0</maxForceRev>
       <maxAngle>${pi/2}</maxAngle>

File: usn_drone_gazebo/urdf/thruster_layouts/usn_drone_t_thrusters.xacro (robot description, xacro)
@@ -13,5 +13,4 @@
       <xacro:usn_drone_gazebo_thruster_config name="left" />
       <xacro:usn_drone_gazebo_thruster_config name="right" />
-      <!-- <xacro:usn_drone_gazebo_thruster_config name="lateral" /> -->
     </plugin>
   </gazebo>

File: usn_drone_gazebo/urdf/usn_drone_gazebo.urdf.xacro (robot description, xacro)
@@ -1,9 +1,8 @@
 <?xml version="1.0"?>
 <!-- Basic WAM-V with gazebo plugins for dynamics -->
-<robot xmlns:xacro="http://ros.org/wiki/xacro"
-       name="WAM-V">
+<robot xmlns:xacro="http://ros.org/wiki/xacro" name="WAM-V">
   <xacro:arg name="locked" default="false" />
   <xacro:arg name="thruster_config" default="H" />
-  <xacro:arg name="camera_enabled" default="false" />
+  <xacro:arg name="camera_enabled" default="true" />
   <xacro:arg name="gps_enabled" default="false" />
   <xacro:arg name="imu_enabled" default="false" />
@@ -13,13 +12,13 @@
   <xacro:arg name="pinger_enabled" default="false" />
   <xacro:arg name="ball_shooter_enabled" default="false" />
-  <xacro:arg name="thruster_namespace" default="thrusters/"/>
-  <xacro:arg name="camera_namespace" default="cameras/"/>
-  <xacro:arg name="zed_namespace" default="zed/"/>
-  <xacro:arg name="sensor_namespace" default="sensors/"/>
-  <xacro:arg name="pinger_namespace" default="pingers/"/>
-  <xacro:arg name="shooter_namespace" default="shooters/"/>
+  <xacro:arg name="thruster_namespace" default="thrusters/" />
+  <xacro:arg name="camera_namespace" default="cameras/" />
+  <xacro:arg name="zed_namespace" default="zed/" />
+  <xacro:arg name="sensor_namespace" default="sensors/" />
+  <xacro:arg name="pinger_namespace" default="pingers/" />
+  <xacro:arg name="shooter_namespace" default="shooters/" />
   <!-- Note: this is only used for some sensors that do not correctly use the
   robotNamespace parameter -->
-  <xacro:arg name="namespace" default="usn_drone"/>
+  <xacro:arg name="namespace" default="usn_drone" />
   <xacro:property name="thruster_namespace" value="$(arg thruster_namespace)" scope="global" />
   <xacro:property name="camera_namespace" value="$(arg camera_namespace)" scope="global" />
@@ -29,11 +28,11 @@
   <xacro:property name="namespace" value="$(arg namespace)" scope="global" />
   <!-- Sensor yaml file -->
-  <xacro:arg name="yaml_component_generation" default="false"/>
-  <xacro:arg name="component_xacro_file" default = ""/>
+  <xacro:arg name="yaml_component_generation" default="false" />
+  <xacro:arg name="component_xacro_file" default="" />
   <!-- Thruster yaml file -->
-  <xacro:arg name="yaml_thruster_generation" default="false"/>
-  <xacro:arg name="thruster_xacro_file" default = ""/>
+  <xacro:arg name="yaml_thruster_generation" default="false" />
+  <xacro:arg name="thruster_xacro_file" default="" />
   <!-- === The WAM-V platform === -->
-  <xacro:include filename="$(find usn_drone_gazebo)/urdf/usn_drone_gazebo.xacro"/>
+  <xacro:include filename="$(find usn_drone_gazebo)/urdf/usn_drone_gazebo.xacro" />
   <!-- === Batteries === >
   <xacro:include filename="$(find usn_drone_description)/urdf/battery.xacro"/>
@@ -43,20 +42,20 @@
   <!-- Use thruster yaml file if given -->
   <xacro:if value="$(arg yaml_thruster_generation)">
-    <xacro:usn_drone_gazebo thruster_layout="$(arg thruster_xacro_file)"/>
+    <xacro:usn_drone_gazebo thruster_layout="$(arg thruster_xacro_file)" />
   </xacro:if>
   <!-- Otherwise, add thrusters based on thruster_config variable -->
   <xacro:unless value="$(arg yaml_thruster_generation)">
-    <xacro:property name="thruster_conf" value="$(arg thruster_config)"/>
+    <xacro:property name="thruster_conf" value="$(arg thruster_config)" />
     <!-- Default WAM-V with two aft thrusters -->
     <xacro:if value="${thruster_conf == 'H'}">
-       <xacro:usn_drone_gazebo thruster_layout="$(find usn_drone_gazebo)/urdf/thruster_layouts/usn_drone_aft_thrusters.xacro"/>
+      <xacro:usn_drone_gazebo thruster_layout="$(find usn_drone_gazebo)/urdf/thruster_layouts/usn_drone_aft_thrusters.xacro" />
     </xacro:if>
     <!-- usn_drone with "T" thruster configuration -->
     <xacro:if value="${thruster_conf == 'T'}">
-      <xacro:usn_drone_gazebo thruster_layout="$(find usn_drone_gazebo)/urdf/thruster_layouts/usn_drone_t_thrusters.xacro"/>
+      <xacro:usn_drone_gazebo thruster_layout="$(find usn_drone_gazebo)/urdf/thruster_layouts/usn_drone_t_thrusters.xacro" />
     </xacro:if>
     <!-- usn_drone with "X" thruster configuration -->
     <xacro:if value="${thruster_conf == 'X'}">
-      <xacro:usn_drone_gazebo thruster_layout="$(find usn_drone_gazebo)/urdf/thruster_layouts/usn_drone_x_thrusters.xacro"/>
+      <xacro:usn_drone_gazebo thruster_layout="$(find usn_drone_gazebo)/urdf/thruster_layouts/usn_drone_x_thrusters.xacro" />
     </xacro:if>
   </xacro:unless>
@@ -64,5 +63,5 @@
   <xacro:if value="$(arg locked)">
     <gazebo>
-      <link name="usn_drone_external_link"/>
+      <link name="usn_drone_external_link" />
       <joint name="usn_drone_external_pivot_joint" type="universal">
         <parent>usn_drone::usn_drone/base_link</parent>
@@ -91,5 +90,5 @@
   <!-- Use sensor yaml file if given -->
   <xacro:if value="$(arg yaml_component_generation)">
-    <xacro:include filename="$(arg component_xacro_file)"/>
+    <xacro:include filename="$(arg component_xacro_file)" />
     <xacro:yaml_components />
     <!-- Add CPU Cases >
@@ -101,5 +100,5 @@
     <!-- Add a front camera -->
     <xacro:if value="$(arg camera_enabled)">
-      <xacro:usn_drone_camera name="front_camera" y="0.3" x="0.75" P="${radians(15)}" />
+      <xacro:usn_drone_camera name="front_camera" y="0" x="0.175" z="0.225" P="${radians(15)}" />
     </xacro:if>
     <!-- <xacro:usn_drone_camera name="zed" y="0" x="2" P="${radians(15)}" /> -->
@@ -114,9 +113,9 @@
     <!-- Add 3D LIDAR -->
     <xacro:if value="$(arg lidar_enabled)">
-      <xacro:lidar name="lidar_usn_drone" y="-0.3" type="16_beam"/>
+      <xacro:lidar name="lidar_usn_drone" y="-0.3" type="16_beam" />
     </xacro:if>
     <!-- Add P3D ground truth -->
     <xacro:if value="$(arg ground_truth_enabled)">
-      <xacro:usn_drone_p3d name="p3d_usn_drone"/>
+      <xacro:usn_drone_p3d name="p3d_usn_drone" />
     </xacro:if>
     <!-- Add pinger -->
@@ -126,5 +125,5 @@
     <!-- Add ball shooter (default pitch angle: ~-60 deg) -->
     <xacro:if value="$(arg ball_shooter_enabled)">
-      <xacro:usn_drone_ball_shooter name="ball_shooter" x="0.54" y="0.30" z="1.296" pitch="-1.04"/>
+      <xacro:usn_drone_ball_shooter name="ball_shooter" x="0.54" y="0.30" z="1.296" pitch="-1.04" />
     </xacro:if>
     <!-- ==== VRX sensor configuration ==== -->
@@ -134,5 +133,5 @@
       <xacro:cpu_cases position="-0.15 0 1.53" orientation="0 0 0"/-->
       <!-- Add a stereo camera pair -->
-      <xacro:usn_drone_camera name="front_left_camera" y="0.1" x="0.75" P="${radians(15)}" />
+      <!-- <xacro:usn_drone_camera name="front_left_camera" y="0.1" x="0.75" P="${radians(15)}" /> -->
       <!-- <xacro:usn_drone_camera name="front_right_camera" y="-0.1" x="0.75" P="${radians(15)}" /> -->
       <!-- Add a camera facing right >

File: wamv_gazebo/urdf/thruster_layouts/wamv_gazebo_thruster_config.xacro (robot description, xacro)
@@ -13,6 +13,6 @@
       <mappingType>1</mappingType>
       <maxCmd>1.0</maxCmd>
-      <maxForceFwd>250.0</maxForceFwd>
-      <maxForceRev>-100.0</maxForceRev>
+      <maxForceFwd>0.0</maxForceFwd>
+      <maxForceRev>0.0</maxForceRev>
       <maxAngle>${pi/2}</maxAngle>
     </thruster>

File: wave_gazebo/world_models/ocean_waves/model.xacro (robot description, xacro)
@@ -17,6 +17,6 @@
 -->
 <world xmlns:xacro="http://ros.org/wiki/xacro">
-  <xacro:macro name="ocean_waves" params="gain:=0.1 period:=5
-                     direction_x:=1.0 direction_y:=0.0
+  <xacro:macro name="ocean_waves" params="gain:=0 period:=5
+                     direction_x:=0 direction_y:=0.0
                      angle:=0.4 scale:=1.5">
   <model name='ocean_waves'>
