Commit message: minor rviz and xacro changes

File: usn_drone_gazebo/urdf/components/usn_drone_imu.xacro (robot description, xacro)
@@ -1,9 +1,5 @@
 <?xml version="1.0"?>
 <robot xmlns:xacro="http://ros.org/wiki/xacro">
-<<<<<<< HEAD:usn_drone_gazebo/urdf/components/usn_drone_imu.xacro
   <xacro:macro name="usn_drone_imu" params="name:=imu x:=0 y:=0 z:=0 R:=0 P:=0 Y:=0 update_rate:=15">
-=======
-  <xacro:macro name="wamv_imu" params="name:=imu x:=0 y:=0 z:=0 R:=0 P:=0 Y:=0 update_rate:=15">
->>>>>>> master:usn_drone_gazebo/urdf/components/wamv_imu.xacro
     <link name="${namespace}/${name}_link">
       <visual name="${name}_visual">>

File: usn_drone_gazebo/urdf/usn_drone_gazebo.urdf.xacro (robot description, xacro)
@@ -109,9 +109,5 @@
     <!-- Add Simulated IMU -->
     <xacro:if value="$(arg imu_enabled)">
-<<<<<<< HEAD
       <xacro:usn_drone_imu name="imu_usn_drone" />
-=======
-      <xacro:wamv_imu name="imu_wamv" />
->>>>>>> master
     </xacro:if>
     <!-- Add 3D LIDAR -->
@@ -137,5 +133,4 @@
       <xacro:cpu_cases position="-0.15 0 1.53" orientation="0 0 0"/-->
       <!-- Add a stereo camera pair -->
-<<<<<<< HEAD
       <!-- <xacro:usn_drone_camera name="front_left_camera" y="0.1" x="0.75" P="${radians(15)}" /> -->
       <!-- <xacro:usn_drone_camera name="front_right_camera" y="-0.1" x="0.75" P="${radians(15)}" /> -->
@@ -146,20 +141,8 @@
       <!-- Add Simulated IMU -->
       <xacro:usn_drone_imu name="imu_usn_drone" x="-0.05" z="0.0" />
-=======
-      <!-- Add a camera facing right >
-      <xacro:wamv_camera name="middle_right_camera" y="-0.45" P="${radians(15)}" Y="${radians(-90)}" post_Y="${radians(-90)}" /-->
-      <!-- Add simulated GPS -->
-      <xacro:wamv_gps name="gps_wamv" x="0.05" z="0.0" />
-      <!-- Add Simulated IMU -->
-      <xacro:wamv_imu name="imu_wamv" x="-0.05" z="0.0" />
->>>>>>> master
       <!-- Add 3D LIDAR -->
       <xacro:lidar name="lidar_usn_drone" type="16_beam" />
       <!-- Add pinger >
-<<<<<<< HEAD
       <xacro:usn_drone_pinger name="pinger" position="1.0 0 -1.0" /-->
-=======
-      <xacro:wamv_pinger name="pinger" position="1.0 0 -1.0" /-->
->>>>>>> master
       <!-- Add ball shooter (default pitch angle: ~-60 deg) >
       <xacro:usn_drone_ball_shooter name="ball_shooter" x="0.54" y="0.30" z="1.296" pitch="-1.04"/-->
@@ -178,7 +161,3 @@
     </plugin>
   </gazebo>
-<<<<<<< HEAD
 </robot>
-=======
-</robot>
->>>>>>> master

File: wave_gazebo/world_models/ocean_waves/model.xacro (robot description, xacro)
@@ -17,13 +17,7 @@
 -->
 <world xmlns:xacro="http://ros.org/wiki/xacro">
-<<<<<<< HEAD
   <xacro:macro name="ocean_waves" params="gain:=0 period:=5
                      direction_x:=0 direction_y:=0.0
-                     angle:=0.4 scale:=1.5">
-=======
-  <xacro:macro name="ocean_waves" params="gain:=1 period:=3
-                     direction_x:=1.0 direction_y:=0.0
-                     angle:=0.4 scale:=1">
->>>>>>> master
+                     angle:=0.4 scale:=0">
   <model name='ocean_waves'>
     <static>true</static>
