Commit message: changed wind and wave parameters

File: vrx_gazebo/worlds/example_course.world.xacro (robot description, xacro)
@@ -7,5 +7,5 @@
     <!--Waves-->
     <xacro:include filename="$(find wave_gazebo)/world_models/ocean_waves/model.xacro"/>
-    <xacro:ocean_waves scale="2.5"/>
+    <xacro:ocean_waves scale="1.5"/>
     <!--Wind-->
     <xacro:include filename="$(find vrx_gazebo)/worlds/xacros/usv_wind_plugin.xacro"/>
@@ -15,5 +15,5 @@
           <name>usn_drone</name>
           <link_name>usn_drone/base_link</link_name>
-          <coeff_vector>.5 .5 .33</coeff_vector>
+          <coeff_vector>.1 .1 .06</coeff_vector>
         </wind_obj>
       </wind_objs>

File: vrx_gazebo/worlds/xacros/usv_wind_plugin.xacro (robot description, xacro)
@@ -4,6 +4,6 @@
                params="**wind_objs
                          direction:=270.0
-                         mean_vel:=20.0
-                         var_gain:=20.0
+                         mean_vel:=1
+                         var_gain:=5
                          var_time:=2.0
                          seed:=''

File: wave_gazebo/world_models/ocean_waves/model.xacro (robot description, xacro)
@@ -17,5 +17,5 @@
 -->
 <world xmlns:xacro="http://ros.org/wiki/xacro">
-  <xacro:macro name="ocean_waves" params="gain:=0.1 period:=5
+  <xacro:macro name="ocean_waves" params="gain:=0.3 period:=5
                      direction_x:=1.0 direction_y:=0.0
                      angle:=0.4 scale:=1.5">
