Commit message: changed dynamics and parameters, test mpc

File: usn_drone_description/urdf/thrusters/engine.xacro (robot description, xacro)
@@ -22,5 +22,5 @@
       </collision>
       <inertial>
-        <mass value="15"/>
+        <mass value="0.15"/>
         <inertia ixx="0.889245" ixy="0.0" ixz="0.0" iyy="0.911125" iyz="0.0" izz="0.078125"/>
       </inertial>
@@ -39,5 +39,5 @@
       </collision>
       <inertial>
-        <mass value="0.5"/>
+        <mass value="0.2"/>
         <inertia ixx="0.008545" ixy="0.0" ixz="0.0" iyy="0.008545" iyz="0.0" izz="0.0144"/>
       </inertial>

File: usn_drone_gazebo/urdf/dynamics/usn_drone_gazebo_dynamics_plugin.xacro (robot description, xacro)
@@ -1,5 +1,5 @@
 <?xml version="1.0"?>
 <robot xmlns:xacro="http://ros.org/wiki/xacro">
-  <xacro:macro name="usv_dynamics_gazebo" params="name width:=2.4 length:=4.9">
+  <xacro:macro name="usv_dynamics_gazebo" params="name width:=0.3 length:=1.8">
     <!--Gazebo Plugin for simulating WAM-V dynamics-->
     <gazebo>
@@ -10,17 +10,17 @@
         <waterDensity>997.8</waterDensity>
         <!-- Added mass -->
-        <xDotU>5.0</xDotU>
-        <yDotV>5.0</yDotV>
-        <nDotR>1.0</nDotR>
+        <xDotU>0.0</xDotU>
+        <yDotV>0.0</yDotV>
+        <nDotR>0.0</nDotR>
         <!-- Linear and quadratic drag -->
-        <xU>51.3</xU>
-        <xUU>72.4</xUU>
-        <yV>40.0</yV>
+        <xU>20.3</xU>
+        <xUU>0.0</xUU>
+        <yV>20.0</yV>
         <yVV>0.0</yVV>
-        <zW>500.0</zW>
-        <kP>50.0</kP>
-        <mQ>50.0</mQ>
-        <nR>400.0</nR>
-        <nRR>0.0</nRR>
+        <zW>20.0</zW>
+        <kP>20.0</kP>
+        <mQ>20.0</mQ>
+        <nR>20.0</nR>
+        <nRR>20.0</nRR>
         <!-- General dimensions -->
         <!--<boatArea>2.2</boatArea>-->

File: usn_drone_gazebo/urdf/thruster_layouts/usn_drone_gazebo_thruster_config.xacro (robot description, xacro)
@@ -13,6 +13,6 @@
       <mappingType>1</mappingType>
       <maxCmd>1</maxCmd>
-      <maxForceFwd>100</maxForceFwd>
-      <maxForceRev>-100.0</maxForceRev>
+      <maxForceFwd>36.297</maxForceFwd>
+      <maxForceRev>-28.449</maxForceRev>
       <maxAngle>${pi/2}</maxAngle>
     </thruster>

File: usn_drone_gazebo/urdf/thruster_layouts/usn_drone_t_thrusters.xacro (robot description, xacro)
@@ -2,6 +2,6 @@
 <robot xmlns:xacro="http://ros.org/wiki/xacro">
   <xacro:include filename="$(find usn_drone_description)/urdf/thrusters/engine.xacro" />
-  <xacro:engine prefix="left" position="-0.5 0.2 0.0" />
-  <xacro:engine prefix="right" position="-0.5 -0.2 0.0" />
+  <xacro:engine prefix="left" position="-0.5 0.14 0.0" />
+  <xacro:engine prefix="right" position="-0.5 -0.14 0.0" />
   <!-- <xacro:engine prefix="lateral" position="0.0 0.0 0.318237" orientation="0.0 0.0 1.5707"/> -->
   <gazebo>

File: vrx_gazebo/worlds/xacros/usv_wind_plugin.xacro (robot description, xacro)
@@ -4,10 +4,10 @@
                params="**wind_objs
                          direction:=0
-                         mean_vel:= 0
-                         var_gain:=0
+                         mean_vel:= 2
+                         var_gain:=1
                          var_time:=2.0
                          seed:=''
                          ros_update_rate:=10
-                         topic_wind_speed:=/vrx/debug/wind/speed
+                         topic_wind_speed:=/vrx/debug/wind/speed123
                          topic_wind_direction:=/vrx/debug/wind/direction
                          " >
@@ -17,10 +17,10 @@
       <xacro:insert_block name="wind_objs"/>
       <!-- Wind -->
-      <wind_direction>${direction}</wind_direction> <!-- in degrees -->
-      <wind_mean_velocity>${mean_vel}</wind_mean_velocity>
-      <var_wind_gain_constants>${var_gain}</var_wind_gain_constants>
-      <var_wind_time_constants>${var_time}</var_wind_time_constants>
-      <random_seed>${seed}</random_seed> <!-- set to zero/empty to randomize -->
-      <update_rate>${ros_update_rate}</update_rate>
+      <wind_direction>0</wind_direction> <!-- in degrees -->
+      <wind_mean_velocity>2</wind_mean_velocity>
+      <var_wind_gain_constants>1</var_wind_gain_constants>
+      <var_wind_time_constants>2</var_wind_time_constants>
+      <random_seed>0</random_seed> <!-- set to zero/empty to randomize -->
+      <update_rate>10</update_rate>
       <topic_wind_speed>${topic_wind_speed}</topic_wind_speed>
       <topic_wind_direction>${topic_wind_direction}</topic_wind_direction>

File: wamv_gazebo/urdf/thruster_layouts/wamv_gazebo_thruster_config.xacro (robot description, xacro)
@@ -13,6 +13,6 @@
       <mappingType>1</mappingType>
       <maxCmd>1.0</maxCmd>
-      <maxForceFwd>0.0</maxForceFwd>
-      <maxForceRev>0.0</maxForceRev>
+      <maxForceFwd>250.0</maxForceFwd>
+      <maxForceRev>-100</maxForceRev>
       <maxAngle>${pi/2}</maxAngle>
     </thruster>

File: wave_gazebo/world_models/ocean_waves/model.xacro (robot description, xacro)
@@ -17,6 +17,6 @@
 -->
 <world xmlns:xacro="http://ros.org/wiki/xacro">
-  <xacro:macro name="ocean_waves" params="gain:=0 period:=5
-                     direction_x:=0 direction_y:=0.0
+  <xacro:macro name="ocean_waves" params="gain:=0.18 period:=1
+                     direction_x:=1.0 direction_y:=0.0
                      angle:=0.4 scale:=1.5">
   <model name='ocean_waves'>
