Commit message: merge

File: gazebo/wave_gazebo/world_models/ocean_waves/model.xacro (robot description, xacro)
@@ -17,7 +17,7 @@
 -->
 <world xmlns:xacro="http://ros.org/wiki/xacro">
-  <xacro:macro name="ocean_waves" params="gain:=0 period:=5
-                     direction_x:=0 direction_y:=0.0
-                     angle:=0.4 scale:=0">
+  <xacro:macro name="ocean_waves" params="gain:=0.18 period:=1
+                     direction_x:=1.0 direction_y:=0.0
+                     angle:=0.4 scale:=1.5">
   <model name='ocean_waves'>
     <static>true</static>
