Commit message: added usn_colreg package with moving boats

File: gazebo/vrx_gazebo/worlds/example_course.world.xacro (robot description, xacro)
@@ -9,5 +9,5 @@
     <xacro:ocean_waves scale="1"/>
     <!--Wind-->
-    <!-- <xacro:include filename="$(find vrx_gazebo)/worlds/xacros/usv_wind_plugin.xacro"/>
+    <xacro:include filename="$(find vrx_gazebo)/worlds/xacros/usv_wind_plugin.xacro"/>
     <xacro:usv_wind_gazebo>
       <wind_objs>
@@ -18,5 +18,5 @@
         </wind_obj>
       </wind_objs>
-    </xacro:usv_wind_gazebo> -->
+    </xacro:usv_wind_gazebo>
     <!-- The light buoy -->
     <include>

File: usn_drone_description/urdf/usn_drone.urdf (robot description, URDF)
Before this commit: robot usn_drone, 1 links, 0 joints
Links:
- link usn_drone/base_link: geometry collision mesh filename=package://usn_drone_description/meshes/usn_drone.STL; visual mesh filename=package://usn_drone_description/meshes/usn_drone.STL

File: usn_drone_gazebo/urdf/components/lidar.xacro (robot description, xacro)
@@ -5,5 +5,5 @@
                params = "type:='16_beam'
                          name
-                         x:=0.7 y:=0 z:=0.1
+                         x:=0.7 y:=0 z:=0.02
                          R:=0 P:=0 Y:=0
                          post_Y:=0 post_z_from:=0">

File: usn_drone_gazebo/urdf/components/usn_drone_camera.xacro (robot description, xacro)
@@ -125,8 +125,6 @@
         </camera>
         <plugin name="camera_plugin" filename="libgazebo_ros_openni_kinect.so">
-          <baseline>0.2</baseline>
+          <baseline>0.12</baseline>
           <alwaysOn>true</alwaysOn>
-          <!-- Keep this zero, update_rate in the parent <sensor> tag
-            will control the frame rate. -->
           <updateRate>0.0</updateRate>
           <cameraName>camera_ir</cameraName>
@@ -147,5 +145,5 @@
           <Cx>0</Cx>
           <Cy>0</Cy>
-          <focalLength>0</focalLength>
+          <focalLength>0.212</focalLength>
           <hackBaseline>0</hackBaseline>
         </plugin>

File: usn_drone_gazebo/urdf/thruster_layouts/usn_drone_gazebo_thruster_config.xacro (robot description, xacro)
@@ -11,8 +11,8 @@
       <enableAngle>${enable_angle}</enableAngle>
       <!-- Optional Parameters -->
-      <mappingType>1</mappingType>
+      <mappingType>0</mappingType>
       <maxCmd>1</maxCmd>
       <maxForceFwd>28.449</maxForceFwd>
-      <maxForceRev>-20</maxForceRev>
+      <maxForceRev>28.449</maxForceRev>
       <maxAngle>${pi/2}</maxAngle>
     </thruster>

File: usn_drone_gazebo/urdf/usn_drone_gazebo.urdf.xacro (robot description, xacro)
@@ -100,5 +100,5 @@
     <!-- Add a front camera -->
     <xacro:if value="$(arg camera_enabled)">
-      <xacro:usn_drone_camera name="front_camera" y="0" x="0.175" z="0.225" P="${radians(15)}" />
+      <xacro:usn_drone_camera name="front_camera" y="0" x="0.175" z="0.4" P="${radians(15)}" />
     </xacro:if>
     <!-- <xacro:usn_drone_camera name="zed" y="0" x="2" P="${radians(15)}" /> -->
@@ -113,5 +113,5 @@
     <!-- Add 3D LIDAR -->
     <xacro:if value="$(arg lidar_enabled)">
-      <xacro:lidar name="lidar_usn_drone" y="-0.3" type="16_beam" />
+      <xacro:lidar name="lidar_usn_drone" y="-0.3" z="-0.2" type="16_beam" />
     </xacro:if>
     <!-- Add P3D ground truth -->
@@ -136,5 +136,5 @@
       <!-- <xacro:usn_drone_camera name="front_right_camera" y="-0.1" x="0.75" P="${radians(15)}" /> -->
       <!-- <Add a camera facing right > -->
-      <xacro:wamv_camera name="front_camera_color" y="0.065" x="0.175" z="0.225" P="${radians(15)}" />
+      <!--xacro:wamv_camera name="front_camera_color" y="0.065" x="0.175" z="0.225" P="${radians(15)}" /-->
       <!-- Add simulated GPS -->
       <xacro:usn_drone_gps name="gps_usn_drone" x="0.05" z="0.0" />

Commit message: more testing and plotting

File: gazebo/vrx_gazebo/worlds/example_course.world.xacro (robot description, xacro)
@@ -7,5 +7,5 @@
     <!--Waves-->
     <xacro:include filename="$(find wave_gazebo)/world_models/ocean_waves/model.xacro"/>
-    <xacro:ocean_waves scale="1"/>
+    <xacro:ocean_waves scale="2"/>
     <!--Wind-->
     <xacro:include filename="$(find vrx_gazebo)/worlds/xacros/usv_wind_plugin.xacro"/>
@@ -15,5 +15,5 @@
           <name>usn_drone</name>
           <link_name>usn_drone/base_link</link_name>
-          <coeff_vector>.1 .1 .06</coeff_vector>
+          <coeff_vector>.2 .2 .12</coeff_vector>
         </wind_obj>
       </wind_objs>

File: gazebo/vrx_gazebo/worlds/xacros/usv_wind_plugin.xacro (robot description, xacro)
@@ -5,6 +5,6 @@
                          direction:=0
                          mean_vel:= 0
-                         var_gain:=0
-                         var_time:=2.0
+                         var_gain:=10
+                         var_time:=1
                          seed:=''
                          ros_update_rate:=10
@@ -19,5 +19,5 @@
       <wind_direction>0</wind_direction> <!-- in degrees -->
       <wind_mean_velocity>0</wind_mean_velocity>
-      <var_wind_gain_constants>1</var_wind_gain_constants>
+      <var_wind_gain_constants>2.3</var_wind_gain_constants>
       <var_wind_time_constants>2</var_wind_time_constants>
       <random_seed>0</random_seed> <!-- set to zero/empty to randomize -->

File: gazebo/wave_gazebo/world_models/ocean_waves/model.xacro (robot description, xacro)
@@ -17,5 +17,5 @@
 -->
 <world xmlns:xacro="http://ros.org/wiki/xacro">
-  <xacro:macro name="ocean_waves" params="gain:=0.18 period:=1
+  <xacro:macro name="ocean_waves" params="gain:=1 period:=1.3
                      direction_x:=1.0 direction_y:=0.0
                      angle:=0.4 scale:=1.5">

Commit message: added heron_pid_ctrl for experimentation

File: gazebo/vrx_gazebo/worlds/example_course.world.xacro (robot description, xacro)
@@ -15,5 +15,7 @@
           <name>usn_drone</name>
           <link_name>usn_drone/base_link</link_name>
+          <!-- uncomment to enable wind impact on boat -->
           <coeff_vector>.2 .2 .12</coeff_vector>
+          <!-- <coeff_vector>0 0 0</coeff_vector> -->
         </wind_obj>
       </wind_objs>

File: gazebo/wave_gazebo/world_models/ocean_waves/model.xacro (robot description, xacro)
@@ -17,5 +17,5 @@
 -->
 <world xmlns:xacro="http://ros.org/wiki/xacro">
-  <xacro:macro name="ocean_waves" params="gain:=1 period:=1.3
+  <xacro:macro name="ocean_waves" params="gain:=1.5 period:=1.3
                      direction_x:=1.0 direction_y:=0.0
                      angle:=0.4 scale:=1.5">

File: usn_drone/usn_drone_gazebo/urdf/thruster_layouts/usn_drone_gazebo_thruster_config.xacro (robot description, xacro)
@@ -13,5 +13,5 @@
       <mappingType>1</mappingType>
       <maxCmd>1</maxCmd>
-      <maxForceFwd>28</maxForceFwd>
+      <maxForceFwd>20</maxForceFwd>
       <maxForceRev>-20</maxForceRev>
       <maxAngle>${pi/2}</maxAngle>
